Commit message: split launch files to work with hardware and sim

File: packages/high_level_control/sentry/sentry_urdf/urdf/sentry_base.urdf.xacro (robot description, xacro)
@@ -3,5 +3,5 @@
   xmlns:xacro="http://www.ros.org/wiki/xacro"
   xmlns:interface="http://playerstage.sourceforge.net/gazebo/xmlschema/#interface">
-  <xacro:property name="wheel_size_y" value="${bodywidth/2}" />
+  <xacro:property name="wheel_size_y" value="0.197" />
   <xacro:property name="wheel_radius" value="0.085" />
   <xacro:property name="wheel_offset_y" value="${bodywidth/2 + wheel_size_y/2}" />
@@ -10,7 +10,7 @@
   <!-- define the base-link origin to lie at floor level, between the drive wheels-->
    <!--main body is a simple box; origin is a center of box-->
-  <xacro:property name="bodylen" value="1.0" />
-  <xacro:property name="bodywidth" value="0.5" />
-  <xacro:property name="bodyheight" value="1.2" />
+  <xacro:property name="bodylen" value="1.22" />
+  <xacro:property name="bodywidth" value="0.368" />
+  <xacro:property name="bodyheight" value="1.346" />
   <xacro:property name="default_mass" value="1.0" />
   <xacro:property name="lidar_cube_size" value="0.25" />

Commit message: changed dimensions

File: packages/high_level_control/sentry/sentry_urdf/urdf/sentry_base.urdf.xacro (robot description, xacro)
@@ -10,9 +10,9 @@
   <!-- define the base-link origin to lie at floor level, between the drive wheels-->
    <!--main body is a simple box; origin is a center of box-->
-  <xacro:property name="bodylen" value="1.22" />
+  <xacro:property name="bodylen" value="1.068" />
   <xacro:property name="bodywidth" value="0.368" />
   <xacro:property name="bodyheight" value="1.346" />
   <xacro:property name="default_mass" value="1.0" />
-  <xacro:property name="lidar_cube_size" value="0.25" />
+  <xacro:property name="lidar_cube_size" value="0.152" />
   <xacro:property name="lidar_dist_up_body" value="0.2" />
   <!-- "track" is the distance between the wheels -->

Commit message: semi jank hector

File: packages/high_level_control/sentry/sentry_urdf/urdf/sentry_base.urdf.xacro (robot description, xacro)
@@ -15,5 +15,5 @@
   <xacro:property name="default_mass" value="1.0" />
   <xacro:property name="lidar_cube_size" value="0.152" />
-  <xacro:property name="lidar_dist_up_body" value="0.2" />
+  <xacro:property name="lidar_dist_from_ground" value="0.32" />
   <!-- "track" is the distance between the wheels -->
   <xacro:property name="track" value=".52" />
@@ -106,5 +106,5 @@
     <joint name="lidar_joint" type="fixed">
         <axis xyz="0 1 0" />
-        <origin xyz="${bodylen/2 + lidar_cube_size/2} 0 ${lidar_dist_up_body - bodylen/2}" rpy="0 0 0"/>
+        <origin xyz="${bodylen/2 + lidar_cube_size/2} 0 ${lidar_dist_from_ground + lidar_cube_size/2 - bodyheight/2 - wheel_radius}" rpy="0 0 0"/>
         <parent link="base_link"/>
         <child link="lidar_link"/>

Commit message: updated launch files and sentry urdf with kinect

File: packages/high_level_control/sentry/sentry_urdf/urdf/sentry_base.urdf.xacro (robot description, xacro)
@@ -142,4 +142,79 @@
       </sensor>
     </gazebo>
+	<!-- add a simulated Kinect camera, including visual, collision and inertial properties, and physics simulation-->
+	<link name="kinect_link">
+      <!-- here is the physical body (case) of the camera-->
+      <collision>
+          <origin xyz="0 0 0" rpy="0 0 0"/>
+          <geometry>
+              <box size="0.02 0.1 0.02"/>
+          </geometry>
+      </collision>
+      <visual>
+          <origin xyz="0 0 0" rpy="0 0 0" />
+          <geometry>
+              <box size="0.02 0.1 0.02"/>
+          </geometry>
+          <material name="camera_case">
+              <color rgba="0.0 0.0 0.7 1.0"/>
+          </material>
+      </visual>
+      <inertial>
+          <mass value="0.1" />
+          <origin xyz="0 0 0" rpy="0 0 0"/>
+          <inertia ixx="0.0001" ixy="0" ixz="0" iyy="0.0001" iyz="0" izz="0.0001" />
+      </inertial>
+  </link>
+  <joint name="kinect_joint" type="fixed">
+    	<parent link="base_link" />
+    	<child link="kinect_link" />
+    	<origin rpy="0 0 0 " xyz="${bodylen/2} 0 ${bodyheight/2}"/>
+    </joint>
+    <!-- kinect depth frame has a different viewpoint; publish it separately-->
+ 	<!-- here is the gazebo plug-in to simulate a color camera -->
+ 	<!--must refer to the above-defined link to place the camera in space-->
+  <gazebo reference="kinect_link">
+    <sensor type="depth" name="openni_camera_camera">
+        <always_on>1</always_on>
+        <visualize>true</visualize>
+        <camera>
+            <horizontal_fov>1.047</horizontal_fov>
+            <image>
+                <width>640</width>
+                <height>480</height>
+                <format>R8G8B8</format>
+            </image>
+            <depth_camera>
+            </depth_camera>
+            <clip>
+                <near>0.1</near>
+                <far>100</far>
+            </clip>
+        </camera>
+      <!--here is the plug-in that does the work of kinect emulation-->
+       <plugin name="camera_controller" filename="libgazebo_ros_openni_kinect.so">
+            <alwaysOn>true</alwaysOn>
+                <updateRate>10.0</updateRate>
+                <cameraName>kinect</cameraName>
+                <frameName>kinect_depth_frame</frameName>
+            <imageTopicName>rgb/image_raw</imageTopicName>
+            <depthImageTopicName>depth/image_raw</depthImageTopicName>
+            <pointCloudTopicName>depth/points</pointCloudTopicName>
+            <cameraInfoTopicName>rgb/camera_info</cameraInfoTopicName>
+            <depthImageCameraInfoTopicName>depth/camera_info</depthImageCameraInfoTopicName>
+            <pointCloudCutoff>0.4</pointCloudCutoff>
+                <hackBaseline>0.07</hackBaseline>
+                <distortionK1>0.0</distortionK1>
+                <distortionK2>0.0</distortionK2>
+                <distortionK3>0.0</distortionK3>
+                <distortionT1>0.0</distortionT1>
+                <distortionT2>0.0</distortionT2>
+            <CxPrime>0.0</CxPrime>
+            <Cx>0.0</Cx>
+            <Cy>0.0</Cy>
+            <focalLength>0.0</focalLength>
+            </plugin>
+    </sensor>
+  </gazebo>
     <xacro:tracked_wheel parent="base_link" prefix="left_0" offset_x= "${2*wheel_spacing}" offset_y = "${wheel_offset_y}" offset_z = "${wheel_offset_z_from_base_link}"/>
     <xacro:tracked_wheel parent="base_link" prefix="left_1" offset_x= "0.0" offset_y = "${wheel_offset_y}" offset_z = "${wheel_offset_z_from_base_link}"/>

Commit message: added simulation terrain world and kinect processing

File: packages/high_level_control/sentry/sentry_urdf/urdf/sentry_base.urdf.xacro (robot description, xacro)
@@ -12,5 +12,5 @@
   <xacro:property name="bodylen" value="1.068" />
   <xacro:property name="bodywidth" value="0.368" />
-  <xacro:property name="bodyheight" value="1.346" />
+  <xacro:property name="bodyheight" value="0.914" />
   <xacro:property name="default_mass" value="1.0" />
   <xacro:property name="lidar_cube_size" value="0.152" />
@@ -180,5 +180,5 @@
         <camera>
             <!-- original: <horizontal_fov>1.047</horizontal_fov> -->
-            <horizontal_fov>2.36</horizontal_fov>
+            <horizontal_fov>1.571</horizontal_fov>
             <image>
                 <width>640</width>
@@ -189,6 +189,6 @@
             </depth_camera>
             <clip>
-                <near>0.1</near>
-                <far>100</far>
+                <near>0.02</near>
+                <far>300</far>
             </clip>
         </camera>
@@ -224,10 +224,10 @@
     <xacro:tracked_wheel parent="base_link" prefix="left_4" offset_x= "${-wheel_spacing}" offset_y = "${wheel_offset_y}" offset_z = "${wheel_offset_z_from_base_link}"/>
     <!-- additional left wheels -->
-    <!-- <xacro:tracked_wheel parent="base_link" prefix="left_5" offset_x= "${-3*wheel_spacing}" offset_y = "${wheel_offset_y}" offset_z = "${wheel_offset_z_from_base_link}"/>
+    <xacro:tracked_wheel parent="base_link" prefix="left_5" offset_x= "${-3*wheel_spacing}" offset_y = "${wheel_offset_y}" offset_z = "${wheel_offset_z_from_base_link}"/>
     <xacro:tracked_wheel parent="base_link" prefix="left_6" offset_x= "${3*wheel_spacing}" offset_y = "${wheel_offset_y}" offset_z = "${wheel_offset_z_from_base_link}"/>
     <xacro:tracked_wheel parent="base_link" prefix="left_7" offset_x= "${-4*wheel_spacing}" offset_y = "${wheel_offset_y}" offset_z = "${wheel_offset_z_from_base_link}"/>
     <xacro:tracked_wheel parent="base_link" prefix="left_8" offset_x= "${4*wheel_spacing}" offset_y = "${wheel_offset_y}" offset_z = "${wheel_offset_z_from_base_link}"/>
     <xacro:tracked_wheel parent="base_link" prefix="left_9" offset_x= "${-5*wheel_spacing}" offset_y = "${wheel_offset_y}" offset_z = "${wheel_offset_z_from_base_link}"/>
-    <xacro:tracked_wheel parent="base_link" prefix="left_10" offset_x= "${5*wheel_spacing}" offset_y = "${wheel_offset_y}" offset_z = "${wheel_offset_z_from_base_link}"/> -->
+    <xacro:tracked_wheel parent="base_link" prefix="left_10" offset_x= "${5*wheel_spacing}" offset_y = "${wheel_offset_y}" offset_z = "${wheel_offset_z_from_base_link}"/>
     <xacro:tracked_wheel parent="base_link" prefix="right_0" offset_x= "${2*wheel_spacing}" offset_y = "-${wheel_offset_y}" offset_z = "${wheel_offset_z_from_base_link}"/>
     <xacro:tracked_wheel parent="base_link" prefix="right_1" offset_x= "0.0" offset_y = "-${wheel_offset_y}" offset_z = "${wheel_offset_z_from_base_link}"/>
@@ -236,10 +236,10 @@
     <xacro:tracked_wheel parent="base_link" prefix="right_4" offset_x= "${wheel_spacing}" offset_y = "-${wheel_offset_y}" offset_z = "${wheel_offset_z_from_base_link}"/>
     <!-- additional right wheels -->
-    <!-- <xacro:tracked_wheel parent="base_link" prefix="right_5" offset_x= "${-3*wheel_spacing}" offset_y = "-${wheel_offset_y}" offset_z = "${wheel_offset_z_from_base_link}"/>
+     <xacro:tracked_wheel parent="base_link" prefix="right_5" offset_x= "${-3*wheel_spacing}" offset_y = "-${wheel_offset_y}" offset_z = "${wheel_offset_z_from_base_link}"/>
     <xacro:tracked_wheel parent="base_link" prefix="right_6" offset_x= "${3*wheel_spacing}" offset_y = "-${wheel_offset_y}" offset_z = "${wheel_offset_z_from_base_link}"/>
     <xacro:tracked_wheel parent="base_link" prefix="right_7" offset_x= "${-4*wheel_spacing}" offset_y = "-${wheel_offset_y}" offset_z = "${wheel_offset_z_from_base_link}"/>
     <xacro:tracked_wheel parent="base_link" prefix="right_8" offset_x= "${4*wheel_spacing}" offset_y = "-${wheel_offset_y}" offset_z = "${wheel_offset_z_from_base_link}"/>
     <xacro:tracked_wheel parent="base_link" prefix="right_9" offset_x= "${-5*wheel_spacing}" offset_y = "-${wheel_offset_y}" offset_z = "${wheel_offset_z_from_base_link}"/>
-    <xacro:tracked_wheel parent="base_link" prefix="right_10" offset_x= "${5*wheel_spacing}" offset_y = "-${wheel_offset_y}" offset_z = "${wheel_offset_z_from_base_link}"/> -->
+    <xacro:tracked_wheel parent="base_link" prefix="right_10" offset_x= "${5*wheel_spacing}" offset_y = "-${wheel_offset_y}" offset_z = "${wheel_offset_z_from_base_link}"/>
     <gazebo>
       <plugin name="diffdrive_plugin_multiwheel" filename="libdiffdrive_plugin_multi_wheel.so">
